Commit message: Detecte and publish the target object pose

File: kuka_kr6_description/urdf/kuka_kr6r900sixx.xacro (robot description, xacro)
@@ -119,5 +119,13 @@
     </link>
     <!-- This frame corresponds to the $FLANGE coordinate system in KUKA KRC controllers. -->
-    <link name="tool0"/>
+    <link name="tool0">
+        <xacro:default_inertial mass = '0.000000001'/>
+        <visual>
+            <origin xyz = '0 0 0.05' rpy = '0 0 0'/>
+            <geometry>
+                <box size = "0.08 0.08 0.08" />
+            </geometry>
+        </visual>
+    </link>
     <!--############################################################################################-->
         <!--Definition of robot's joints-->

File: kuka_kr6_description/urdf/sensors/camera.gazebo.xacro (robot description, xacro)
@@ -4,5 +4,5 @@
     <material>Gazebo/Red</material>
     <sensor name="camera" type="depth">
-      <update_rate>20</update_rate>
+      <update_rate>30.0</update_rate>
       <camera>
         <horizontal_fov>1.047198</horizontal_fov>

File: kuka_kr6_description/urdf/sensors/camera.urdf.xacro (robot description, xacro)
@@ -5,5 +5,5 @@
   <xacro:property name="CAM_RADIUS" value="0.05" />
    <joint name="camera_joint" type="fixed">
-        <origin xyz="1.5 0 1.0" rpy="${PI} ${5*PI/6} 0"/>
+        <origin xyz="1.15 0 0.7" rpy="${PI} ${3/4*PI} 0"/>
         <parent link="base_link"/>
         <child link="camera_link"/>
@@ -27,7 +27,8 @@
       <origin xyz="0 0 0" rpy="0 0 0"/>
       <geometry>
-        <cylinder length="${CAM_LEN}" radius="${CAM_RADIUS}"/>
+        <!--<cylinder length="${CAM_LEN}" radius="${CAM_RADIUS}"/> -->
+        <mesh filename="package://kuka_kr6_description/meshes/camera/kinect.dae"/>
       </geometry>
-      <material name="red"/>
+      <material name="black"/>
     </visual>
     <sensor name="camera" type="depth">

Commit message: Add the obstacles with information published from gazebo

File: kuka_kr6_description/urdf/kuka_kr6r900sixx.xacro (robot description, xacro)
@@ -143,5 +143,6 @@
         <child link="link_2"/>
         <axis xyz="0 1 0"/>
-        <limit effort="0" lower="${-DEG2RAD * 190}" upper="${DEG2RAD * 45}" velocity="${DEG2RAD * 300}"/>
+        <!-- IMPORTANT: The original value here 'upper' is ${DEG2RAD * 45} -->
+        <limit effort="0" lower="${-DEG2RAD * 190}" upper="${DEG2RAD * 75}" velocity="${DEG2RAD * 300}"/>
     </joint>
     <joint name="joint_a3" type="revolute">

File: kuka_kr6_description/urdf/sensors/camera.urdf.xacro (robot description, xacro)
@@ -48,4 +48,10 @@
     </sensor>
   </link>
+   <joint name="camera_joint_vision" type="fixed">
+        <origin xyz="0 0 0" rpy="${-PI/2} 0 ${-PI/2}"/>
+        <parent link="camera_link"/>
+        <child link="camera_vision_link"/>
+   </joint>
+  <link name="camera_vision_link" />
   <xacro:include filename="$(find kuka_kr6_description)/urdf/sensors/camera.gazebo.xacro"/>
 </robot>
