Commit message: modified some RRT functions

File: kuka_kr6_description/urdf/kuka_arm.xacro (robot description, xacro)
@@ -4,8 +4,9 @@
     <xacro:include filename="$(find kuka_kr6_description)/urdf/sensors/camera.urdf.xacro"/>
     <xacro:include filename="$(find kuka_kr6_description)/urdf/kuka_kr6r900sixx.xacro"/>
+    <!--<xacro:include filename="$(find kuka_kr6_description)/urdf/gripper.xacro"/>-->
     <link name="world"/>
     <joint name="world_joint" type="fixed">
         <parent link="world" />
-        <child link = "base_link" />
+        <child link="base_link" />
         <origin xyz="0 0 0." rpy="0.0 0.0 0.0" />
     </joint>

File: kuka_kr6_description/urdf/kuka_kr6r900sixx.xacro (robot description, xacro)
@@ -121,10 +121,10 @@
     <link name="tool0">
         <xacro:default_inertial mass = '0.000000001'/>
-        <visual>
+        <!--<visual>
             <origin xyz = '0 0 0.05' rpy = '0 0 0'/>
             <geometry>
                 <box size = "0.08 0.08 0.08" />
             </geometry>
-        </visual>
+        </visual>-->
     </link>
     <!--############################################################################################-->
